File: Cube-Panel.brd (EAGLE design)
At the start: 100 x 100 mm, 126 parts

Commit message: Rerouted power-traces for LEDs so the with increased from 0.75mm to 1.5mm
Parts:
- added R4: (no value), _Passive:R1206
- moved R3 20.9 mm to (-10.2, 2.54), turned to 0 degrees
- moved R1 16.1 mm to (-7.62, -2.54), turned to 0 degrees
- moved R2 16.1 mm to (-7.62, 2.54), turned to 0 degrees
- moved C1 0.79 mm to (-39.5, -44.5)
- moved C10 0.79 mm to (-2.00, -32.0)
- moved C11 0.79 mm to (2.00, -30.5)
- moved C12 0.79 mm to (14.5, -30.5)
- moved C13 0.79 mm to (-39.5, -19.5)
- moved C14 0.79 mm to (-27.0, -19.5)
- moved C15 0.79 mm to (-14.5, -19.5)
- moved C16 0.79 mm to (-2.00, -19.5)
- moved C17 0.79 mm to (2.00, -18.0)
- moved C18 0.79 mm to (14.5, -18.0)
- moved C19 0.79 mm to (27.0, -18.0)
- moved C2 0.79 mm to (-27.0, -44.5)
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Routing:
- net GND: track 947.6 -> 915.6 mm
- net VCC: track 914.7 -> 887.0 mm
