File: Cube-Panel.sch (EAGLE design)
At the start: 126 parts

Commit message: Rerouted power-traces for LEDs so the with increased from 0.75mm to 1.5mm
Parts:
- added R4: (no value), _Passive:WIDERSTAND_1206
Changed lines of the file:
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@@
 <part name="R2" library="_Passive" deviceset="WIDERSTAND" device="_0603"/>
 <part name="R3" library="_Passive" deviceset="WIDERSTAND" device="_0603"/>
+<part name="R4" library="_Passive" deviceset="WIDERSTAND" device="_1206"/>
 </parts>
 <sheets>
@@
 <instance part="R2" gate="G$1" x="-53.34" y="40.64" rot="R90"/>
 <instance part="R3" gate="G$1" x="-53.34" y="30.48" rot="R90"/>
+<instance part="R4" gate="G$1" x="-55.88" y="152.4"/>
 </instances>
 <busses>
