File: pcb/Cube-Panel.sch (EAGLE design)
At the start: 139 parts, among them IC1 MBI5041-GP, IC2 ATTINY(261/461/861)V-MAZ

Commit message: Added resistors (0603) for path-configurability.
Parts:
- added R10, R100, R101, R102, R103, R104, R105, R106, R107, R108, R109, R11, R110, R111, R112, R113, R114, R115, R116, R117, R118, R119, R12, R120, R121, R122, R123, R124, R125, R126, R127, R128, R129, R13, R130, R131, R132, R133, R134, R135, R136, R137, R138, R139, R14, R140, R141, R142, R143, R144, R145, R146, R147, R148, R149, R15, R150, R151, R152, R153, R154, R155, R156, R157, R158, R159, R16, R160, R161, R162, R163, R164, R165, R166, R167, R168, R169, R17, R170, R171, R172, R173, R174, R175, R176, R177, R178, R179, R18, R180, R181, R182, R183, R184, R185, R186, R187, R188, R189, R19, R190, R191, R192, R193, R194, R195, R196, R197, R198, R199, R20, R200, R201, R202, R203, R204, R205, R206, R207, R208, R209, R21, R210, R211, R212, R213, R214, R215, R22, R23, R24, R25, R26, R27, R28, R29, R30, R31, R32, R33, R34, R35, R36, R37, R38, R39, R40, R41, R42, R43, R44, R45, R46, R47, R48, R49, R50, R51, R52, R53, R54, R55, R56, R57, R58, R59, R60, R61, R62, R63, R64, R65, R66, R67, R68, R69, R7, R70, R71, R72, R73, R74, R75, R76, R77, R78, R79, R8, R80, R81, R82, R83, R84, R85, R86, R87, R88, R89, R9, R90, R91, R92, R93, R94, R95, R96, R97, R98, R99: (no value), _Passive:WIDERSTAND-0603
Connections:
- new net IN1: LED1.DIN, R13.2, R15.2
- new net IN10: LED10.DIN, R23.2, R39.2, R46.2, R73.2
- new net IN11: LED11.DIN, R31.2, R42.2, R50.2, R77.2
- new net IN12: LED12.DIN, R45.2, R49.2, R81.2
- new net IN13: LED13.DIN, R14.2, R24.2, R54.2
- new net IN14: LED14.DIN, R10.2, R34.2, R65.2, R90.2
- new net IN15: LED15.DIN, R109.2, R21.2, R27.2, R71.2
- new net IN16: LED16.DIN, R113.2, R29.2, R70.2, R75.2
- new net IN17: LED17.DIN, R117.2, R47.2, R74.2, R79.2
- new net IN18: LED18.DIN, R121.2, R51.2, R78.2, R83.2
- new net IN19: LED19.DIN, R125.2, R82.2, R87.2
- new net IN2: LED2.DIN, R11.2, R28.2, R35.2
- new net IN20: LED20.DIN, R129.2, R86.2
- new net IN21: LED21.DIN, R32.2, R57.2, R85.2
- new net IN22: LED22.DIN, R107.2, R25.2, R55.2, R94.2
- new net IN23: LED23.DIN, R111.2, R132.2, R68.2, R91.2
- new net IN24: LED24.DIN, R110.2, R115.2, R136.2, R72.2
- new net IN25: LED25.DIN, R114.2, R119.2, R140.2, R76.2
- new net IN26: LED26.DIN, R118.2, R123.2, R144.2, R80.2
- new net IN27: LED27.DIN, R122.2, R127.2, R148.2, R84.2
- new net IN28: LED28.DIN, R126.2, R152.2, R88.2
- new net IN29: LED29.DIN, R53.2, R60.2, R92.2
- new net IN3: LED3.DIN, R19.2, R22.2, R38.2
- new net IN30: LED30.DIN, R130.2, R58.2, R89.2, R98.2
- new net IN31: LED31.DIN, R108.2, R134.2, R155.2, R95.2
- new net IN32: LED32.DIN, R112.2, R133.2, R138.2, R159.2
- new net IN33: LED33.DIN, R116.2, R137.2, R142.2, R163.2
- new net IN34: LED34.DIN, R120.2, R141.2, R146.2, R167.2
- new net IN35: LED35.DIN, R124.2, R145.2, R150.2, R171.2
- new net IN36: LED36.DIN, R128.2, R149.2, R175.2
- new net IN37: LED37.DIN, R56.2, R63.2, R96.2
- new net IN38: LED38.DIN, R102.2, R153.2, R61.2, R93.2
- new net IN39: LED39.DIN, R131.2, R157.2, R178.2, R99.2
- new net IN4: LED4.DIN, R30.2, R37.2, R41.2
- new net IN40: LED40.DIN, R135.2, R156.2, R161.2, R182.2
- new net IN41: LED41.DIN, R139.2, R160.2, R165.2, R186.2
- new net IN42: LED42.DIN, R143.2, R164.2, R169.2, R190.2
- new net IN43: LED43.DIN, R147.2, R168.2, R173.2, R194.2
- new net IN44: LED44.DIN, R151.2, R172.2, R198.2
- new net IN45: LED45.DIN, R100.2, R59.2, R66.2
- new net IN46: LED46.DIN, R105.2, R176.2, R64.2, R97.2
- new net IN47: LED47.DIN, R103.2, R154.2, R180.2, R200.2
- new net IN48: LED48.DIN, R158.2, R179.2, R184.2, R203.2
- new net IN49: LED49.DIN, R162.2, R183.2, R188.2, R206.2
- new net IN5: LED5.DIN, R40.2, R44.2, R48.2
- new net IN50: LED50.DIN, R166.2, R187.2, R192.2, R209.2
- new net IN51: LED51.DIN, R170.2, R191.2, R196.2, R212.2
- new net IN52: LED52.DIN, R174.2, R195.2, R215.2
- new net IN53: LED53.DIN, R104.2, R62.2
- new net IN54: LED54.DIN, R101.2, R199.2, R67.2
- new net IN55: LED55.DIN, R106.2, R177.2, R202.2
- new net IN56: LED56.DIN, R181.2, R201.2, R205.2
- new net IN57: LED57.DIN, R185.2, R204.2, R208.2
- new net IN58: LED58.DIN, R189.2, R207.2, R211.2
- new net IN59: LED59.DIN, R193.2, R210.2, R214.2
- new net IN6: LED6.DIN, R43.2, R52.2
- new net IN60: LED60.DIN, R197.2, R213.2
- new net IN7: LED7.DIN, R18.2, R33.2, R9.2
- new net IN8: LED8.DIN, R16.2, R17.2, R20.2, R26.2
- new net IN9: LED9.DIN, R12.2, R36.2, R4.2, R69.2
- new net OUT1: LED1.DOUT, R18.1, R28.1
- new net OUT10: LED10.DOUT, R29.1, R30.1, R31.1, R4.1
- new net OUT11: LED11.DOUT, R46.1, R47.1, R48.1, R49.1
- new net OUT12: LED12.DOUT, R50.1, R51.1, R52.1
- new net OUT13: LED13.DOUT, R32.1, R33.1, R34.1
- new net OUT14: LED14.DOUT, R24.1, R25.1, R26.1, R27.1
- new net OUT15: LED15.DOUT, R65.1, R68.1, R69.1, R70.1
- new net OUT16: LED16.DOUT, R71.1, R72.1, R73.1, R74.1
- new net OUT17: LED17.DOUT, R75.1, R76.1, R77.1, R78.1
- new net OUT18: LED18.DOUT, R79.1, R80.1, R81.1, R82.1
- new net OUT19: LED19.DOUT, R83.1, R84.1, R86.1
- new net OUT2: LED2.DOUT, R13.1, R17.1, R19.1
- new net OUT20: LED20.DOUT, R87.1, R88.1
- new net OUT21: LED21.DOUT, R53.1, R54.1, R55.1
- new net OUT22: LED22.DOUT, R85.1, R89.1, R90.1, R91.1
- new net OUT23: LED23.DOUT, R107.1, R108.1, R109.1, R110.1
- new net OUT24: LED24.DOUT, R111.1, R112.1, R113.1, R114.1
- new net OUT25: LED25.DOUT, R115.1, R116.1, R117.1, R118.1, R119.1, R120.1, R121.1, R122.1
- new net OUT26: LED26.DOUT, R123.1, R124.1, R125.1, R126.1
- new net OUT27: LED27.DOUT, R127.1, R128.1, R129.1
- new net OUT28: LED28.DOUT
- new net OUT29: LED29.DOUT, R56.1, R57.1, R58.1
- new net OUT3: LED3.DOUT, R35.1, R36.1, R37.1
- new net OUT30: LED30.DOUT, R92.1, R93.1, R94.1, R95.1
- new net OUT31: LED31.DOUT, R130.1, R131.1, R132.1, R133.1
- new net OUT32: LED32.DOUT, R134.1, R135.1, R136.1, R137.1
- new net OUT33: LED33.DOUT, R138.1, R139.1, R140.1, R141.1
- new net OUT34: LED34.DOUT, R142.1, R143.1, R144.1, R145.1
- new net OUT35: LED35.DOUT, R146.1, R147.1, R148.1, R149.1
- new net OUT36: LED36.DOUT, R150.1, R151.1, R152.1
- new net OUT37: LED37.DOUT, R59.1, R60.1, R61.1
- new net OUT38: LED38.DOUT, R96.1, R97.1, R98.1, R99.1
- new net OUT39: LED39.DOUT, R153.1, R154.1, R155.1, R156.1
- new net OUT4: LED4.DOUT, R38.1, R39.1, R40.1
- new net OUT40: LED40.DOUT, R157.1, R158.1, R159.1, R160.1
- new net OUT41: LED41.DOUT, R161.1, R162.1, R163.1, R164.1
- new net OUT42: LED42.DOUT, R165.1, R166.1, R167.1, R168.1
- new net OUT43: LED43.DOUT, R169.1, R170.1, R171.1, R172.1
- new net OUT44: LED44.DOUT, R173.1, R174.1, R175.1
- new net OUT45: LED45.DOUT, R62.1, R63.1, R64.1
- new net OUT46: LED46.DOUT, R100.1, R101.1, R102.1, R103.1
- new net OUT47: LED47.DOUT, R176.1, R177.1, R178.1, R179.1
- new net OUT48: LED48.DOUT, R180.1, R181.1, R182.1, R183.1
- new net OUT49: LED49.DOUT, R184.1, R185.1, R186.1, R187.1
- new net OUT5: LED5.DOUT, R41.1, R42.1, R43.1
- new net OUT50: LED50.DOUT, R188.1, R189.1, R190.1, R191.1
- new net OUT51: LED51.DOUT, R192.1, R193.1, R194.1, R195.1
- new net OUT52: LED52.DOUT, R196.1, R197.1, R198.1
- new net OUT53: LED53.DOUT, R66.1, R67.1
- new net OUT54: LED54.DOUT, R104.1, R105.1, R106.1
- new net OUT55: LED55.DOUT, R199.1, R200.1, R201.1
- new net OUT56: LED56.DOUT, R202.1, R203.1, R204.1
- new net OUT57: LED57.DOUT, R205.1, R206.1, R207.1
- new net OUT58: LED58.DOUT, R208.1, R209.1, R210.1
- new net OUT59: LED59.DOUT, R211.1, R212.1, R213.1
- new net OUT6: LED6.DOUT, R44.1, R45.1
- new net OUT60: LED60.DOUT, R214.1, R215.1
- new net OUT7: LED7.DOUT, R14.1, R15.1, R16.1
- new net OUT8: LED8.DOUT, R10.1, R11.1, R12.1, R9.1
- new net OUT9: LED9.DOUT, R20.1, R21.1, R22.1, R23.1
- net N$26: now also R8.1
- net N$35: now also R7.1
- net VCC: now also R7.2, R8.2

Commit message: Added wired data-path resistors.
Parts:
- removed R1, R2, R3: (no value), _Passive:WIDERSTAND-0603
- removed SV1: (no value), con-lstb:MA10-1
Connections:
- removed net ID: R1.2, R2.2, SV1.3
- removed net N$1: R2.1, R3.2
- net GND: no longer R1.1, R3.1, SV1.1, SV1.2
- net OUT25: no longer R119.1, R120.1, R121.1, R122.1
- net OUT26: now also R119.1, R120.1, R121.1, R122.1; no longer R123.1, R124.1, R125.1, R126.1
- net OUT27: now also R123.1, R124.1, R125.1, R126.1; no longer R127.1, R128.1, R129.1
- net OUT28: now also R127.1, R128.1, R129.1
- net VCC: no longer SV1.10, SV1.9
Changed lines of the file:
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@@
 <part name="GND6" library="supply1" deviceset="GND" device=""/>
 <part name="P+6" library="supply1" deviceset="VCC" device=""/>
-<part name="SV1" library="con-lstb" deviceset="MA10-1" device=""/>
-<part name="P+7" library="supply1" deviceset="VCC" device=""/>
-<part name="GND7" library="supply1" deviceset="GND" device=""/>
 <part name="IC1" library="_ICs" deviceset="MBI5041" device="-GP"/>
 <part name="GND8" library="supply1" deviceset="GND" device=""/>
@@
 <part name="TP5" library="_Messpunkte" deviceset="TP" device=""/>
 <part name="TP6" library="_Messpunkte" deviceset="TP" device=""/>
-<part name="R1" library="_Passive" deviceset="WIDERSTAND" device="-0603"/>
-<part name="R2" library="_Passive" deviceset="WIDERSTAND" device="-0603"/>
-<part name="R3" library="_Passive" deviceset="WIDERSTAND" device="-0603"/>
 <part name="R6" library="_Passive" deviceset="WIDERSTAND" device="-0603"/>
 <part name="R5" library="_Passive" deviceset="WIDERSTAND" device="-0603"/>
@@
 <instance part="GND6" gate="1" x="279.4" y="-12.7"/>
 <instance part="P+6" gate="VCC" x="279.4" y="10.16"/>
-<instance part="SV1" gate="1" x="-50.8" y="0"/>
-<instance part="P+7" gate="VCC" x="-40.64" y="17.78" rot="MR0"/>
-<instance part="GND7" gate="1" x="-40.64" y="-30.48"/>
 <instance part="IC1" gate="G$1" x="304.8" y="58.42"/>
 <instance part="GND8" gate="1" x="271.78" y="40.64"/>
@@
 <instance part="TP5" gate="G$1" x="431.8" y="157.48" rot="R270"/>
 <instance part="TP6" gate="G$1" x="363.22" y="147.32" rot="R90"/>
-<instance part="R1" gate="G$1" x="-33.02" y="-15.24" rot="R90"/>
-<instance part="R2" gate="G$1" x="-27.94" y="-10.16" rot="R90"/>
-<instance part="R3" gate="G$1" x="-27.94" y="-20.32" rot="R90"/>
 <instance part="R6" gate="G$1" x="441.96" y="149.86" rot="R90"/>
 <instance part="R5" gate="G$1" x="271.78" y="50.8" rot="R90"/>
@@
 </segment>
 <segment>
-<pinref part="SV1" gate="1" pin="2"/>
-<wire x1="-43.18" y1="-7.62" x2="-40.64" y2="-7.62" width="0.1524" layer="91"/>
-<wire x1="-40.64" y1="-7.62" x2="-40.64" y2="-10.16" width="0.1524" layer="91"/>
-<pinref part="SV1" gate="1" pin="1"/>
-<wire x1="-40.64" y1="-10.16" x2="-40.64" y2="-25.4" width="0.1524" layer="91"/>
-<wire x1="-40.64" y1="-25.4" x2="-40.64" y2="-27.94" width="0.1524" layer="91"/>
-<wire x1="-43.18" y1="-10.16" x2="-40.64" y2="-10.16" width="0.1524" layer="91"/>
-<junction x="-40.64" y="-10.16"/>
-<pinref part="GND7" gate="1" pin="GND"/>
-<wire x1="-27.94" y1="-25.4" x2="-33.02" y2="-25.4" width="0.1524" layer="91"/>
-<junction x="-40.64" y="-25.4"/>
-<wire x1="-33.02" y1="-25.4" x2="-40.64" y2="-25.4" width="0.1524" layer="91"/>
-<wire x1="-33.02" y1="-20.32" x2="-33.02" y2="-25.4" width="0.1524" layer="91"/>
-<junction x="-33.02" y="-25.4"/>
-<pinref part="R1" gate="G$1" pin="1"/>
-<pinref part="R3" gate="G$1" pin="1"/>
-</segment>
-<segment>
 <pinref part="IC1" gate="G$1" pin="GND"/>
 <wire x1="276.86" y1="45.72" x2="271.78" y2="45.72" width="0.1524" layer="91"/>
@@
 </segment>
 <segment>
-<pinref part="SV1" gate="1" pin="9"/>
-<wire x1="-43.18" y1="10.16" x2="-40.64" y2="10.16" width="0.1524" layer="91"/>
-<wire x1="-40.64" y1="10.16" x2="-40.64" y2="12.7" width="0.1524" layer="91"/>
-<pinref part="SV1" gate="1" pin="10"/>
-<wire x1="-40.64" y1="12.7" x2="-40.64" y2="15.24" width="0.1524" layer="91"/>
-<wire x1="-43.18" y1="12.7" x2="-40.64" y2="12.7" width="0.1524" layer="91"/>
-<junction x="-40.64" y="12.7"/>
-<pinref part="P+7" gate="VCC" pin="VCC"/>
-</segment>
-<segment>
 <pinref part="IC1" gate="G$1" pin="VCC"/>
 <pinref part="P+8" gate="VCC" pin="VCC"/>
@@
 </segment>
 </net>
-<net name="ID" class="0">
-<segment>
-<pinref part="SV1" gate="1" pin="3"/>
-<wire x1="-43.18" y1="-5.08" x2="-33.02" y2="-5.08" width="0.1524" layer="91"/>
-<label x="-42.926" y="-4.826" size="1.27" layer="95"/>
-<wire x1="-33.02" y1="-5.08" x2="-27.94" y2="-5.08" width="0.1524" layer="91"/>
-<wire x1="-33.02" y1="-10.16" x2="-33.02" y2="-5.08" width="0.1524" layer="91"/>
-<junction x="-33.02" y="-5.08"/>
-<pinref part="R1" gate="G$1" pin="2"/>
-<pinref part="R2" gate="G$1" pin="2"/>
-</segment>
-</net>
 <net name="B2" class="0">
 <segment>
@@
 </segment>
 </net>
-<net name="N$1" class="0">
-<segment>
-<pinref part="R2" gate="G$1" pin="1"/>
-<pinref part="R3" gate="G$1" pin="2"/>
-</segment>
-</net>
 </nets>
 </sheet>
@@
 <net name="IN28" class="0">
 <segment>
-<pinref part="R88" gate="G$1" pin="2"/>
-<wire x1="393.7" y1="127" x2="393.7" y2="129.54" width="0.1524" layer="91"/>
-<label x="393.7" y="129.54" size="1.27" layer="95" rot="R90" xref="yes"/>
-</segment>
-<segment>
 <pinref part="R126" gate="G$1" pin="2"/>
 <wire x1="350.52" y1="170.18" x2="353.06" y2="170.18" width="0.1524" layer="91"/>
@@
 <label x="393.7" y="210.82" size="1.27" layer="95" rot="R270" xref="yes"/>
 </segment>
+<segment>
+<pinref part="R88" gate="G$1" pin="2"/>
+<wire x1="393.7" y1="127" x2="393.7" y2="129.54" width="0.1524" layer="91"/>
+<label x="393.7" y="129.54" size="1.27" layer="95" rot="R90" xref="yes"/>
+</segment>
 </net>
 <net name="OUT22" class="0">
@@
 <label x="226.568" y="170.942" size="1.27" layer="95"/>
 </segment>
-<segment>
-<pinref part="R119" gate="G$1" pin="1"/>
-<pinref part="R122" gate="G$1" pin="1"/>
-<wire x1="279.4" y1="170.18" x2="281.94" y2="170.18" width="0.1524" layer="91"/>
-<wire x1="281.94" y1="170.18" x2="284.48" y2="170.18" width="0.1524" layer="91"/>
-<pinref part="R121" gate="G$1" pin="1"/>
-<pinref part="R120" gate="G$1" pin="1"/>
-<wire x1="281.94" y1="172.72" x2="281.94" y2="170.18" width="0.1524" layer="91"/>
-<junction x="281.94" y="170.18"/>
-<wire x1="281.94" y1="167.64" x2="281.94" y2="170.18" width="0.1524" layer="91"/>
-<label x="282.448" y="170.942" size="1.27" layer="95"/>
-</segment>
 </net>
 <net name="IN33" class="0">
@@
 </segment>
 </net>
-<net name="OUT26" class="0">
-<segment>
-<pinref part="R123" gate="G$1" pin="1"/>
-<pinref part="R126" gate="G$1" pin="1"/>
-<wire x1="335.28" y1="170.18" x2="337.82" y2="170.18" width="0.1524" layer="91"/>
-<wire x1="337.82" y1="170.18" x2="340.36" y2="170.18" width="0.1524" layer="91"/>
-<pinref part="R125" gate="G$1" pin="1"/>
-<pinref part="R124" gate="G$1" pin="1"/>
-<wire x1="337.82" y1="172.72" x2="337.82" y2="170.18" width="0.1524" layer="91"/>
-<junction x="337.82" y="170.18"/>
-<wire x1="337.82" y1="167.64" x2="337.82" y2="170.18" width="0.1524" layer="91"/>
-<label x="338.328" y="170.942" size="1.27" layer="95"/>
-</segment>
-</net>
 <net name="IN35" class="0">
 <segment>
@@
 <net name="OUT27" class="0">
 <segment>
-<pinref part="R127" gate="G$1" pin="1"/>
-<wire x1="391.16" y1="170.18" x2="393.7" y2="170.18" width="0.1524" layer="91"/>
-<pinref part="R129" gate="G$1" pin="1"/>
-<pinref part="R128" gate="G$1" pin="1"/>
-<wire x1="393.7" y1="172.72" x2="393.7" y2="170.18" width="0.1524" layer="91"/>
-<junction x="393.7" y="170.18"/>
-<wire x1="393.7" y1="167.64" x2="393.7" y2="170.18" width="0.1524" layer="91"/>
-<label x="394.208" y="170.942" size="1.27" layer="95"/>
+<pinref part="R123" gate="G$1" pin="1"/>
+<pinref part="R126" gate="G$1" pin="1"/>
+<wire x1="335.28" y1="170.18" x2="337.82" y2="170.18" width="0.1524" layer="91"/>
+<wire x1="337.82" y1="170.18" x2="340.36" y2="170.18" width="0.1524" layer="91"/>
+<pinref part="R125" gate="G$1" pin="1"/>
+<pinref part="R124" gate="G$1" pin="1"/>
+<wire x1="337.82" y1="172.72" x2="337.82" y2="170.18" width="0.1524" layer="91"/>
+<junction x="337.82" y="170.18"/>
+<wire x1="337.82" y1="167.64" x2="337.82" y2="170.18" width="0.1524" layer="91"/>
+<label x="338.328" y="170.942" size="1.27" layer="95"/>
 </segment>
 </net>
@@
 </segment>
 </net>
+<net name="OUT28" class="0">
+<segment>
+<pinref part="R127" gate="G$1" pin="1"/>
+<wire x1="391.16" y1="170.18" x2="393.7" y2="170.18" width="0.1524" layer="91"/>
+<pinref part="R129" gate="G$1" pin="1"/>
+<pinref part="R128" gate="G$1" pin="1"/>
+<wire x1="393.7" y1="172.72" x2="393.7" y2="170.18" width="0.1524" layer="91"/>
+<junction x="393.7" y="170.18"/>
+<wire x1="393.7" y1="167.64" x2="393.7" y2="170.18" width="0.1524" layer="91"/>
+<label x="394.208" y="170.942" size="1.27" layer="95"/>
+</segment>
+</net>
+<net name="OUT26" class="0">
+<segment>
+<pinref part="R119" gate="G$1" pin="1"/>
+<pinref part="R122" gate="G$1" pin="1"/>
+<wire x1="279.4" y1="170.18" x2="281.94" y2="170.18" width="0.1524" layer="91"/>
+<wire x1="281.94" y1="170.18" x2="284.48" y2="170.18" width="0.1524" layer="91"/>
+<pinref part="R121" gate="G$1" pin="1"/>
+<pinref part="R120" gate="G$1" pin="1"/>
+<wire x1="281.94" y1="172.72" x2="281.94" y2="170.18" width="0.1524" layer="91"/>
+<junction x="281.94" y="170.18"/>
+<wire x1="281.94" y1="167.64" x2="281.94" y2="170.18" width="0.1524" layer="91"/>
+<label x="282.448" y="170.942" size="1.27" layer="95"/>
+</segment>
+</net>

Commit message: Added some labels and did some minor aesthetic corrections.
Parts:
- added R1, R2, R3: (no value), _Passive:WIDERSTAND-0603
- added X2: JP8ER, jumper:JP8ER
Connections:
- new net BUS-RX: IC2.(DO/ADC1/PCINT1)PA1
- new net BUS-TX: IC2.(SDA/DI/ADC0/PCINT0)PA0
- new net N$1: R2.1, R3.2
- new net N$3: R1.2, R2.2, X2.6
- net GND: now also R1.1, R3.1, X2.7, X2.8
- net VCC: now also X2.1, X2.2
Changed lines of the file:
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@@
 <setting verticaltext="up"/>
 </settings>
-<grid distance="2.2" unitdist="inch" unit="inch" style="lines" multiple="1" display="yes" altdistance="0.01" altunitdist="inch" altunit="inch"/>
+<grid distance="0.1" unitdist="inch" unit="inch" style="lines" multiple="1" display="yes" altdistance="0.01" altunitdist="inch" altunit="inch"/>
 <layers>
 <layer number="1" name="Top" color="4" fill="1" visible="no" active="no"/>
@@
 <part name="R214" library="_Passive" deviceset="WIDERSTAND" device="-0603"/>
 <part name="R215" library="_Passive" deviceset="WIDERSTAND" device="-0603"/>
+<part name="GND7" library="supply1" deviceset="GND" device=""/>
+<part name="P+7" library="supply1" deviceset="VCC" device=""/>
+<part name="R1" library="_Passive" deviceset="WIDERSTAND" device="-0603"/>
+<part name="R2" library="_Passive" deviceset="WIDERSTAND" device="-0603"/>
+<part name="R3" library="_Passive" deviceset="WIDERSTAND" device="-0603"/>
+<part name="X2" library="jumper" deviceset="JP8E" device="R"/>
 </parts>
 <sheets>
@@
 <instance part="P+12" gate="VCC" x="320.04" y="124.46"/>
 <instance part="P+13" gate="VCC" x="363.22" y="124.46"/>
+<instance part="GND7" gate="1" x="-27.94" y="2.54" rot="R90"/>
+<instance part="P+7" gate="VCC" x="-55.88" y="2.54" rot="R90"/>
+<instance part="R1" gate="G$1" x="-30.48" y="-12.7" rot="R270"/>
+<instance part="R2" gate="G$1" x="-35.56" y="-17.78" rot="R270"/>
+<instance part="R3" gate="G$1" x="-35.56" y="-7.62" rot="R270"/>
+<instance part="X2" gate="G$1" x="-43.18" y="7.62"/>
 </instances>
 <busses>
@@
 <pinref part="GND10" gate="1" pin="GND"/>
 </segment>
+<segment>
+<pinref part="GND7" gate="1" pin="GND"/>
+<wire x1="-35.56" y1="5.08" x2="-35.56" y2="2.54" width="0.1524" layer="91"/>
+<wire x1="-35.56" y1="2.54" x2="-33.02" y2="2.54" width="0.1524" layer="91"/>
+<wire x1="-33.02" y1="2.54" x2="-30.48" y2="2.54" width="0.1524" layer="91"/>
+<wire x1="-33.02" y1="5.08" x2="-33.02" y2="2.54" width="0.1524" layer="91"/>
+<junction x="-33.02" y="2.54"/>
+<pinref part="R3" gate="G$1" pin="1"/>
+<wire x1="-35.56" y1="0" x2="-35.56" y2="-2.54" width="0.1524" layer="91"/>
+<pinref part="R1" gate="G$1" pin="1"/>
+<wire x1="-35.56" y1="0" x2="-30.48" y2="0" width="0.1524" layer="91"/>
+<wire x1="-30.48" y1="0" x2="-30.48" y2="-7.62" width="0.1524" layer="91"/>
+<wire x1="-35.56" y1="0" x2="-35.56" y2="2.54" width="0.1524" layer="91"/>
+<junction x="-35.56" y="0"/>
+<junction x="-35.56" y="2.54"/>
+<pinref part="X2" gate="G$1" pin="7"/>
+<pinref part="X2" gate="G$1" pin="8"/>
+</segment>
 </net>
 <net name="VCC" class="0">
@@
 <pinref part="P+13" gate="VCC" pin="VCC"/>
 </segment>
+<segment>
+<pinref part="P+7" gate="VCC" pin="VCC"/>
+<wire x1="-53.34" y1="2.54" x2="-50.8" y2="2.54" width="0.1524" layer="91"/>
+<pinref part="X2" gate="G$1" pin="1"/>
+<wire x1="-50.8" y1="2.54" x2="-50.8" y2="5.08" width="0.1524" layer="91"/>
+<pinref part="X2" gate="G$1" pin="2"/>
+<wire x1="-48.26" y1="5.08" x2="-48.26" y2="2.54" width="0.1524" layer="91"/>
+<wire x1="-48.26" y1="2.54" x2="-50.8" y2="2.54" width="0.1524" layer="91"/>
+<junction x="-50.8" y="2.54"/>
+</segment>
 </net>
 <net name="B2" class="0">
@@
 </segment>
 </net>
+<net name="N$1" class="0">
+<segment>
+<pinref part="R2" gate="G$1" pin="1"/>
+<pinref part="R3" gate="G$1" pin="2"/>
+</segment>
+</net>
+<net name="N$3" class="0">
+<segment>
+<pinref part="R2" gate="G$1" pin="2"/>
+<wire x1="-35.56" y1="-22.86" x2="-35.56" y2="-25.4" width="0.1524" layer="91"/>
+<wire x1="-35.56" y1="-25.4" x2="-30.48" y2="-25.4" width="0.1524" layer="91"/>
+<pinref part="R1" gate="G$1" pin="2"/>
+<wire x1="-30.48" y1="-25.4" x2="-30.48" y2="-17.78" width="0.1524" layer="91"/>
+<wire x1="-35.56" y1="-25.4" x2="-38.1" y2="-25.4" width="0.1524" layer="91"/>
+<junction x="-35.56" y="-25.4"/>
+<wire x1="-38.1" y1="-25.4" x2="-38.1" y2="5.08" width="0.1524" layer="91"/>
+<pinref part="X2" gate="G$1" pin="6"/>
+</segment>
+</net>
+<net name="BUS-TX" class="0">
+<segment>
+<pinref part="IC2" gate="G$1" pin="(SDA/DI/ADC0/PCINT0)PA0"/>
+<wire x1="424.18" y1="185.42" x2="426.72" y2="185.42" width="0.1524" layer="91"/>
+<label x="426.72" y="185.42" size="1.27" layer="95" xref="yes"/>
+</segment>
+</net>
+<net name="BUS-RX" class="0">
+<segment>
+<pinref part="IC2" gate="G$1" pin="(DO/ADC1/PCINT1)PA1"/>
+<wire x1="424.18" y1="182.88" x2="426.72" y2="182.88" width="0.1524" layer="91"/>
+<label x="426.72" y="182.88" size="1.27" layer="95" xref="yes"/>
+</segment>
+</net>
