File: pcb/Cube-Panel.sch (EAGLE design)
At the start: 348 parts, among them IC1 MBI5041-GP, IC2 ATTINY(261/461/861)V-MAZ, X2 JP8ER

Commit message: Added Select-Resistor for LED#1
Parts:
- added R216, R217, R218, R219, R220, R221, R222, R223, R224, R225, R226, R227, R228, R229, R230, R231, R232, R233, R234, R235, R236, R237, R238, R239, R240, R241, R242, R243, R244, R245, R246, R247, R248, R249, R250, R251, R252, R253, R254, R255, R256, R257, R258, R259, R260, R261, R262, R263, R264, R265, R266, R267, R268, R269, R270, R271, R272, R273, R274, R275, R276, R277, R278, R279, R280, R281, R282, R283, R284: (no value), _Passive:WIDERSTAND-0603
Connections:
- new net LED-DATA: R283.1, R284.1, X2.3
- new net N$12: R2.2, R216.1, R217.1, R218.1, R219.1, R220.1, R221.1, R222.1, R223.1
- new net N$22: R224.1, R225.1, R226.1, R227.1, R228.1, R229.1, R230.1, R231.1, R270.2
- new net N$32: R232.1, R233.1, R234.1, R235.1, R236.1, R237.1, R238.1, R239.1, R271.2
- new net N$42: R240.1, R241.1, R242.1, R243.1, R244.1, R245.1, R246.1, R247.1, R282.2
- new net N$5: R2.1, R270.1, R271.1, R282.1, R283.2
- new net N$51: R248.1, R249.1, R250.1, R251.1, R252.1, R253.1, R254.1, R255.1, R281.2
- new net N$60: R256.1, R257.1, R258.1, R259.1, R260.1, R261.1, R262.1, R263.1, R280.2
- new net N$69: R264.1, R265.1, R266.1, R267.1, R268.1, R269.1, R279.2
- new net N$78: R272.1, R273.1, R274.1, R275.1, R276.1, R277.1, R278.2
- new net SLAVE_IN: X2.4
- new net SLAVE_OUT: X2.5
- net IN1: now also R277.2
- net IN10: now also R266.2
- net IN11: now also R265.2
- net IN12: now also R264.2
- net IN13: now also R263.2
- net IN14: now also R262.2
- net IN15: now also R261.2
- net IN16: now also R260.2
- net IN17: now also R259.2
- net IN18: now also R258.2
- net IN19: now also R257.2
- net IN2: now also R276.2
- net IN20: now also R256.2
- net IN21: now also R255.2
- net IN22: now also R254.2
- net IN23: now also R253.2
- net IN24: now also R252.2
- net IN25: now also R251.2
- net IN26: now also R250.2
- net IN27: now also R249.2
- net IN28: now also R248.2
- net IN29: now also R247.2
- net IN3: now also R275.2
- net IN30: now also R246.2
- net IN31: now also R245.2
- net IN32: now also R244.2
- net IN33: now also R243.2
- net IN34: now also R242.2
- net IN35: now also R241.2
- net IN36: now also R240.2
- net IN37: now also R239.2
- net IN38: now also R238.2
- net IN39: now also R237.2
- net IN4: now also R274.2
- net IN40: now also R236.2
- net IN41: now also R235.2
- net IN42: now also R234.2
- net IN43: now also R233.2
- net IN44: now also R232.2
- net IN45: now also R231.2
- net IN46: now also R230.2
- net IN47: now also R229.2
- net IN48: now also R228.2
- net IN49: now also R227.2
- net IN5: now also R273.2
- net IN50: now also R226.2
- net IN51: now also R225.2
- net IN52: now also R224.2
- net IN53: now also R223.2
- net IN54: now also R222.2
- net IN55: now also R221.2
- net IN56: now also R220.2
- net IN57: now also R219.2
- net IN58: now also R218.2
- net IN59: now also R217.2
- net IN6: now also R272.2
- net IN60: now also R216.2
- net IN7: now also R269.2
- net IN8: now also R268.2
- net IN9: now also R267.2
- net N$1: now also R278.1, R279.1, R280.1, R281.1, R284.2; no longer R2.1, R3.2
- net N$3: now also R3.2; no longer R2.2

Commit message: Added Feedback-Trace for LED-Data. µC can now drive the LEDs. Added Single-Wire-UART-Bus for Communication.
Parts:
- added C63: (no value), _Passive:KONDENSATOR-0603
- added Q1: DUAL_BJT_NPN_BIAS-PUMH2, _Transistor:DUAL_BJT_NPN_BIAS-PUMH2
- added R285, R286, R287, R288, R289, R290, R291, R292, R293, R294, R295, R296, R297, R298, R299, R300, R301, R302, R303, R304, R305, R306, R307, R308, R309, R310, R311, R312, R313, R314, R315, R316, R317, R318, R319, R320, R321, R322, R323, R324, R325, R326, R327, R328, R329, R330, R331, R332, R333, R334, R335, R336, R337, R338, R339, R340, R341, R342, R343, R344, R345, R346, R347, R348, R349, R350, R351, R352, R353, R354, R355, R356, R357: (no value), _Passive:WIDERSTAND-0603
Connections:
- removed net BUS-RX: IC2.(DO/ADC1/PCINT1)PA1
- removed net BUS-TX: IC2.(SDA/DI/ADC0/PCINT0)PA0
- removed net N$51: R248.1, R249.1, R250.1, R251.1, R252.1, R253.1, R254.1, R255.1, R281.2
- removed net SLAVE_IN: X2.4
- removed net SLAVE_OUT: X2.5
- new net LED-DATA-OUT: R356.1, R357.1, X2.4
- new net LED-DATA-OUT-UC: R287.1, R328.1, R329.1, R330.1, R331.1, R332.1, R333.1, R334.1, R335.1, R353.2
- new net LED-DATA-UC: R248.1, R249.1, R250.1, R251.1, R252.1, R253.1, R254.1, R255.1, R281.2, R286.1
- new net N$10: R312.1, R313.1, R314.1, R315.1, R316.1, R317.1, R318.1, R319.1, R355.2
- new net N$11: R320.1, R321.1, R322.1, R323.1, R324.1, R325.1, R326.1, R327.1, R354.2
- new net N$14: R336.1, R337.1, R338.1, R339.1, R340.1, R341.1, R352.2
- new net N$15: R342.1, R343.1, R344.1, R345.1, R346.1, R347.1, R351.2
- new net N$16: R351.1, R352.1, R353.1, R354.1, R357.2
- new net N$17: R348.1, R349.1, R350.1, R355.1, R356.2
- new net N$18: Q1.1.C, Q1.2.B, R285.2
- new net N$19: IC2.(AREF/PCINT3)PA3, R287.2
- new net N$6: IC2.(SCL/USCK/INT1/ADC2/PCINT2)PA2, R286.2
- new net N$7: R288.1, R289.1, R290.1, R291.1, R292.1, R293.1, R294.1, R295.1, R348.2
- new net N$8: R296.1, R297.1, R298.1, R299.1, R300.1, R301.1, R302.1, R303.1, R349.2
- new net N$9: R304.1, R305.1, R306.1, R307.1, R308.1, R309.1, R310.1, R311.1, R350.2
- new net SERIAL-BUS: IC2.(SDA/DI/ADC0/PCINT0)PA0, Q1.2.C, X2.5
- new net SERIAL-BUS-TX: IC2.(DO/ADC1/PCINT1)PA1, Q1.1.B
- net GND: now also C63.2, Q1.1.E, Q1.2.E
- net OUT1: now also R347.2
- net OUT10: now also R338.2
- net OUT11: now also R337.2
- net OUT12: now also R336.2
- net OUT13: now also R335.2
- net OUT14: now also R334.2
- net OUT15: now also R333.2
- net OUT16: now also R332.2
- net OUT17: now also R331.2
- net OUT18: now also R330.2
- net OUT19: now also R329.2
- net OUT2: now also R346.2
- net OUT20: now also R328.2
- net OUT21: now also R327.2
- net OUT22: now also R326.2
- net OUT23: now also R325.2
- net OUT24: now also R324.2
- net OUT25: now also R323.2
- net OUT26: now also R322.2
- net OUT27: now also R321.2
- net OUT28: now also R320.2
- net OUT29: now also R319.2
- net OUT3: now also R345.2
- net OUT30: now also R318.2
- net OUT31: now also R317.2
- net OUT32: now also R316.2
- net OUT33: now also R315.2
- net OUT34: now also R314.2
- net OUT35: now also R313.2
- net OUT36: now also R312.2
- net OUT37: now also R311.2
- net OUT38: now also R310.2
- net OUT39: now also R309.2
- net OUT4: now also R344.2
- net OUT40: now also R308.2
- net OUT41: now also R307.2
- net OUT42: now also R306.2
- net OUT43: now also R305.2
- net OUT44: now also R304.2
- net OUT45: now also R303.2
- net OUT46: now also R302.2
- net OUT47: now also R301.2
- net OUT48: now also R300.2
- net OUT49: now also R299.2
- net OUT5: now also R343.2
- net OUT50: now also R298.2
- net OUT51: now also R297.2
- net OUT52: now also R296.2
- net OUT53: now also R295.2
- net OUT54: now also R294.2
- net OUT55: now also R293.2
- net OUT56: now also R292.2
- net OUT57: now also R291.2
- net OUT58: now also R290.2
- net OUT59: now also R289.2
- net OUT6: now also R342.2
- net OUT60: now also R288.2
- net OUT7: now also R341.2
- net OUT8: now also R340.2
- net OUT9: now also R339.2
- net VCC: now also C63.1, R285.1

Commit message: µC can now measure its own ID.
Connections:
- removed net N$3: R1.2, R3.2, X2.6
- new net ID-SENSE: IC2.(XTAL1/CLKI/ADC7/!OC1D!/PCINT12)PB4, R1.2, R3.2, X2.6
Other:
- moved on the sheet: R1
Changed lines of the file:
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@@
 <instance part="GND7" gate="1" x="-27.94" y="2.54" rot="R90"/>
 <instance part="P+7" gate="VCC" x="-55.88" y="2.54" rot="R90"/>
-<instance part="R1" gate="G$1" x="-30.48" y="-12.7" rot="R270"/>
+<instance part="R1" gate="G$1" x="-30.48" y="-7.62" rot="R270"/>
 <instance part="R3" gate="G$1" x="-35.56" y="-7.62" rot="R270"/>
 <instance part="X2" gate="G$1" x="-43.18" y="7.62"/>
@@
 <pinref part="R1" gate="G$1" pin="1"/>
 <wire x1="-35.56" y1="0" x2="-30.48" y2="0" width="0.1524" layer="91"/>
-<wire x1="-30.48" y1="0" x2="-30.48" y2="-7.62" width="0.1524" layer="91"/>
+<wire x1="-30.48" y1="0" x2="-30.48" y2="-2.54" width="0.1524" layer="91"/>
 <wire x1="-35.56" y1="0" x2="-35.56" y2="2.54" width="0.1524" layer="91"/>
 <junction x="-35.56" y="0"/>
@@
 </segment>
 </net>
-<net name="N$3" class="0">
-<segment>
-<wire x1="-35.56" y1="-25.4" x2="-30.48" y2="-25.4" width="0.1524" layer="91"/>
-<pinref part="R1" gate="G$1" pin="2"/>
-<wire x1="-30.48" y1="-25.4" x2="-30.48" y2="-17.78" width="0.1524" layer="91"/>
-<wire x1="-35.56" y1="-25.4" x2="-38.1" y2="-25.4" width="0.1524" layer="91"/>
-<junction x="-35.56" y="-25.4"/>
-<wire x1="-38.1" y1="-25.4" x2="-38.1" y2="5.08" width="0.1524" layer="91"/>
-<pinref part="X2" gate="G$1" pin="6"/>
-<wire x1="-35.56" y1="-25.4" x2="-35.56" y2="-12.7" width="0.1524" layer="91"/>
-<pinref part="R3" gate="G$1" pin="2"/>
-</segment>
-</net>
 <net name="SERIAL-BUS-TX" class="0">
 <segment>
@@
 </segment>
 </net>
+<net name="ID-SENSE" class="0">
+<segment>
+<pinref part="IC2" gate="G$1" pin="(XTAL1/CLKI/ADC7/!OC1D!/PCINT12)PB4"/>
+<wire x1="424.18" y1="152.4" x2="426.72" y2="152.4" width="0.1524" layer="91"/>
+<label x="426.72" y="152.4" size="1.27" layer="95" xref="yes"/>
+</segment>
+<segment>
+<wire x1="-35.56" y1="-15.24" x2="-30.48" y2="-15.24" width="0.1524" layer="91"/>
+<pinref part="R1" gate="G$1" pin="2"/>
+<wire x1="-30.48" y1="-15.24" x2="-30.48" y2="-12.7" width="0.1524" layer="91"/>
+<wire x1="-35.56" y1="-15.24" x2="-38.1" y2="-15.24" width="0.1524" layer="91"/>
+<junction x="-35.56" y="-15.24"/>
+<wire x1="-38.1" y1="-15.24" x2="-38.1" y2="5.08" width="0.1524" layer="91"/>
+<pinref part="X2" gate="G$1" pin="6"/>
+<wire x1="-35.56" y1="-15.24" x2="-35.56" y2="-12.7" width="0.1524" layer="91"/>
+<pinref part="R3" gate="G$1" pin="2"/>
+<label x="-38.1" y="-17.018" size="1.27" layer="95"/>
+</segment>
+</net>
